File: IRBeacon/schematics/IRBeaconRev4.brd (EAGLE design)
At the start: 90 x 14.8 mm, 14 parts, among them IC1 LD117AS33TR, SW1 416131160808, X1 53048-06

Commit message: EnkelFugl and some circuit changes
Parts:
- moved C2 14.9 mm to (40.2, 11.4), turned to 270 degrees
- moved C3 1.52 mm to (27.0, 10.6)
Routing:
- net GND: track 27.3 -> 4.56 mm
- net VCC: track 89.3 -> 71.5 mm
- net N$3: track 22.0 -> 20.9 mm
Other:
- board text added: "IRBeacon Rev4"
- board text removed: "IRBeacon Rev 5"
