File: IRBeacon/schematics/IRBeaconRev4.sch (EAGLE design)
At the start: 14 parts, among them IC1 LD117AS33TR, SW1 416131160808, X1 53048-06

Commit message: More pinne fix and circuit stuff
Connections:
- removed net N$11: SW1.9, U$1.(PCINT7/ICP/OC0B/ADC7)PA7
- removed net N$14: SW1.11, U$1.(PCINT5/OC1B/MISO/DO/ADC5)PA5, X1-2.S
- new net N$16: SW1.16, U$1.(PCINT7/ICP/OC0B/ADC7)PA7
- new net N$9: SW1.9, U$1.(PCINT0/AREF/ADC0)PA0
- net N$10: now also SW1.15; no longer SW1.10
- net N$12: now also SW1.14, U$1.(PCINT5/OC1B/MISO/DO/ADC5)PA5, X1-2.S; no longer SW1.16, U$1.(PCINT0/AREF/ADC0)PA0
- net N$4: now also SW1.12, U$1.(PCINT3/T0/ADC3)PA3; no longer SW1.15, U$1.(PCINT1/AIN0/ADC1)PA1
- net N$5: now also SW1.11; no longer SW1.14
- net N$6: now also SW1.10, U$1.(PCINT1/AIN0/ADC1)PA1; no longer SW1.13, U$1.(PCINT3/T0/ADC3)PA3
- net N$8: now also SW1.13; no longer SW1.12
Other:
- moved on the sheet: SW1
Changed lines of the file:
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@@
 <classes>
 <class number="0" name="default" width="0.508" drill="0.508">
-<clearance class="0" value="0.508"/>
+<clearance class="0" value="0.762"/>
 </class>
 </classes>
@@
 </plain>
 <instances>
-<instance part="SW1" gate="G$1" x="81.28" y="40.64"/>
+<instance part="SW1" gate="G$1" x="81.28" y="44.45"/>
 <instance part="U$1" gate="G$1" x="33.02" y="81.28"/>
 <instance part="X1" gate="-1" x="66.04" y="119.38" rot="R90"/>
@@
 <segment>
 <pinref part="GND2" gate="1" pin="GND"/>
-<wire x1="63.5" y1="36.83" x2="63.5" y2="25.4" width="0.1524" layer="91"/>
+<wire x1="63.5" y1="40.64" x2="63.5" y2="25.4" width="0.1524" layer="91"/>
 <wire x1="63.5" y1="25.4" x2="63.5" y2="22.86" width="0.1524" layer="91"/>
-<wire x1="68.58" y1="36.83" x2="68.58" y2="25.4" width="0.1524" layer="91"/>
+<wire x1="68.58" y1="40.64" x2="68.58" y2="25.4" width="0.1524" layer="91"/>
 <wire x1="68.58" y1="25.4" x2="63.5" y2="25.4" width="0.1524" layer="91"/>
 <junction x="63.5" y="25.4"/>
-<wire x1="73.66" y1="36.83" x2="73.66" y2="25.4" width="0.1524" layer="91"/>
+<wire x1="73.66" y1="40.64" x2="73.66" y2="25.4" width="0.1524" layer="91"/>
 <wire x1="73.66" y1="25.4" x2="68.58" y2="25.4" width="0.1524" layer="91"/>
 <junction x="68.58" y="25.4"/>
-<wire x1="78.74" y1="36.83" x2="78.74" y2="25.4" width="0.1524" layer="91"/>
+<wire x1="78.74" y1="40.64" x2="78.74" y2="25.4" width="0.1524" layer="91"/>
 <wire x1="78.74" y1="25.4" x2="73.66" y2="25.4" width="0.1524" layer="91"/>
 <junction x="73.66" y="25.4"/>
-<wire x1="83.82" y1="36.83" x2="83.82" y2="25.4" width="0.1524" layer="91"/>
+<wire x1="83.82" y1="40.64" x2="83.82" y2="25.4" width="0.1524" layer="91"/>
 <wire x1="83.82" y1="25.4" x2="78.74" y2="25.4" width="0.1524" layer="91"/>
 <junction x="78.74" y="25.4"/>
-<wire x1="88.9" y1="36.83" x2="88.9" y2="25.4" width="0.1524" layer="91"/>
+<wire x1="88.9" y1="40.64" x2="88.9" y2="25.4" width="0.1524" layer="91"/>
 <wire x1="88.9" y1="25.4" x2="83.82" y2="25.4" width="0.1524" layer="91"/>
 <junction x="83.82" y="25.4"/>
-<wire x1="93.98" y1="36.83" x2="93.98" y2="25.4" width="0.1524" layer="91"/>
+<wire x1="93.98" y1="40.64" x2="93.98" y2="25.4" width="0.1524" layer="91"/>
 <wire x1="93.98" y1="25.4" x2="88.9" y2="25.4" width="0.1524" layer="91"/>
 <junction x="88.9" y="25.4"/>
-<wire x1="99.06" y1="36.83" x2="99.06" y2="25.4" width="0.1524" layer="91"/>
+<wire x1="99.06" y1="40.64" x2="99.06" y2="25.4" width="0.1524" layer="91"/>
 <wire x1="99.06" y1="25.4" x2="93.98" y2="25.4" width="0.1524" layer="91"/>
 <junction x="93.98" y="25.4"/>
@@
 <net name="N$12" class="0">
 <segment>
-<pinref part="U$1" gate="G$1" pin="(PCINT0/AREF/ADC0)PA0"/>
-<wire x1="58.42" y1="66.04" x2="63.5" y2="66.04" width="0.1524" layer="91"/>
-<pinref part="SW1" gate="G$1" pin="16"/>
-<wire x1="63.5" y1="44.45" x2="63.5" y2="66.04" width="0.1524" layer="91"/>
-</segment>
-</net>
-<net name="N$4" class="0">
-<segment>
-<pinref part="U$1" gate="G$1" pin="(PCINT1/AIN0/ADC1)PA1"/>
-<wire x1="58.42" y1="68.58" x2="68.58" y2="68.58" width="0.1524" layer="91"/>
-<wire x1="68.58" y1="68.58" x2="68.58" y2="44.45" width="0.1524" layer="91"/>
-<pinref part="SW1" gate="G$1" pin="15"/>
-</segment>
-</net>
-<net name="N$5" class="0">
-<segment>
-<pinref part="U$1" gate="G$1" pin="(PCINT2/AIN1/ADC2)PA2"/>
-<wire x1="58.42" y1="71.12" x2="73.66" y2="71.12" width="0.1524" layer="91"/>
-<wire x1="73.66" y1="71.12" x2="73.66" y2="44.45" width="0.1524" layer="91"/>
+<pinref part="U$1" gate="G$1" pin="(PCINT5/OC1B/MISO/DO/ADC5)PA5"/>
+<pinref part="X1" gate="-2" pin="S"/>
+<wire x1="58.42" y1="78.74" x2="68.58" y2="78.74" width="0.1524" layer="91"/>
+<wire x1="68.58" y1="116.84" x2="68.58" y2="78.74" width="0.1524" layer="91"/>
 <pinref part="SW1" gate="G$1" pin="14"/>
-</segment>
-</net>
-<net name="N$6" class="0">
-<segment>
-<pinref part="U$1" gate="G$1" pin="(PCINT3/T0/ADC3)PA3"/>
-<wire x1="58.42" y1="73.66" x2="78.74" y2="73.66" width="0.1524" layer="91"/>
-<wire x1="78.74" y1="73.66" x2="78.74" y2="44.45" width="0.1524" layer="91"/>
-<pinref part="SW1" gate="G$1" pin="13"/>
+<wire x1="73.66" y1="48.26" x2="73.66" y2="78.74" width="0.1524" layer="91"/>
+<wire x1="73.66" y1="78.74" x2="68.58" y2="78.74" width="0.1524" layer="91"/>
+<junction x="68.58" y="78.74"/>
 </segment>
 </net>
@@
 <pinref part="U$1" gate="G$1" pin="(PCINT4/T1/SCL/USCK/ADC4)PA4"/>
 <wire x1="58.42" y1="76.2" x2="76.2" y2="76.2" width="0.1524" layer="91"/>
-<wire x1="76.2" y1="76.2" x2="83.82" y2="76.2" width="0.1524" layer="91"/>
-<wire x1="83.82" y1="76.2" x2="83.82" y2="44.45" width="0.1524" layer="91"/>
-<pinref part="SW1" gate="G$1" pin="12"/>
 <pinref part="X1" gate="-5" pin="S"/>
 <wire x1="76.2" y1="116.84" x2="76.2" y2="76.2" width="0.1524" layer="91"/>
+<pinref part="SW1" gate="G$1" pin="13"/>
+<wire x1="78.74" y1="48.26" x2="78.74" y2="76.2" width="0.1524" layer="91"/>
+<wire x1="78.74" y1="76.2" x2="76.2" y2="76.2" width="0.1524" layer="91"/>
 <junction x="76.2" y="76.2"/>
 </segment>
@@
 <net name="N$10" class="0">
 <segment>
-<wire x1="58.42" y1="81.28" x2="71.12" y2="81.28" width="0.1524" layer="91"/>
-<wire x1="71.12" y1="81.28" x2="93.98" y2="81.28" width="0.1524" layer="91"/>
-<wire x1="93.98" y1="81.28" x2="93.98" y2="44.45" width="0.1524" layer="91"/>
-<pinref part="SW1" gate="G$1" pin="10"/>
+<wire x1="58.42" y1="81.28" x2="66.04" y2="81.28" width="0.1524" layer="91"/>
 <pinref part="U$1" gate="G$1" pin="(PCINT6/OC1A/SDA/MOSI/ADC6)PA6"/>
 <pinref part="X1" gate="-3" pin="S"/>
+<wire x1="66.04" y1="81.28" x2="71.12" y2="81.28" width="0.1524" layer="91"/>
 <wire x1="71.12" y1="116.84" x2="71.12" y2="81.28" width="0.1524" layer="91"/>
-<junction x="71.12" y="81.28"/>
-</segment>
-</net>
-<net name="N$11" class="0">
-<segment>
-<pinref part="U$1" gate="G$1" pin="(PCINT7/ICP/OC0B/ADC7)PA7"/>
-<wire x1="58.42" y1="83.82" x2="99.06" y2="83.82" width="0.1524" layer="91"/>
-<wire x1="99.06" y1="83.82" x2="99.06" y2="44.45" width="0.1524" layer="91"/>
-<pinref part="SW1" gate="G$1" pin="9"/>
+<pinref part="SW1" gate="G$1" pin="15"/>
+<wire x1="68.58" y1="48.26" x2="68.58" y2="63.5" width="0.1524" layer="91"/>
+<wire x1="68.58" y1="63.5" x2="66.04" y2="63.5" width="0.1524" layer="91"/>
+<wire x1="66.04" y1="63.5" x2="66.04" y2="81.28" width="0.1524" layer="91"/>
+<junction x="66.04" y="81.28"/>
 </segment>
 </net>
@@
 <wire x1="114.3" y1="86.36" x2="114.3" y2="81.28" width="0.1524" layer="91"/>
 <pinref part="R2" gate="G$1" pin="1"/>
-</segment>
-</net>
-<net name="N$14" class="0">
-<segment>
-<pinref part="U$1" gate="G$1" pin="(PCINT5/OC1B/MISO/DO/ADC5)PA5"/>
-<wire x1="58.42" y1="78.74" x2="68.58" y2="78.74" width="0.1524" layer="91"/>
-<wire x1="68.58" y1="78.74" x2="88.9" y2="78.74" width="0.1524" layer="91"/>
-<wire x1="88.9" y1="78.74" x2="88.9" y2="44.45" width="0.1524" layer="91"/>
-<pinref part="SW1" gate="G$1" pin="11"/>
-<pinref part="X1" gate="-2" pin="S"/>
-<wire x1="68.58" y1="116.84" x2="68.58" y2="78.74" width="0.1524" layer="91"/>
-<junction x="68.58" y="78.74"/>
 </segment>
 </net>
@@
 </segment>
 </net>
+<net name="N$9" class="0">
+<segment>
+<pinref part="U$1" gate="G$1" pin="(PCINT0/AREF/ADC0)PA0"/>
+<pinref part="SW1" gate="G$1" pin="9"/>
+<wire x1="58.42" y1="66.04" x2="99.06" y2="66.04" width="0.1524" layer="91"/>
+<wire x1="99.06" y1="66.04" x2="99.06" y2="48.26" width="0.1524" layer="91"/>
+</segment>
+</net>
+<net name="N$6" class="0">
+<segment>
+<pinref part="SW1" gate="G$1" pin="10"/>
+<wire x1="93.98" y1="48.26" x2="93.98" y2="68.58" width="0.1524" layer="91"/>
+<pinref part="U$1" gate="G$1" pin="(PCINT1/AIN0/ADC1)PA1"/>
+<wire x1="93.98" y1="68.58" x2="58.42" y2="68.58" width="0.1524" layer="91"/>
+</segment>
+</net>
+<net name="N$5" class="0">
+<segment>
+<pinref part="U$1" gate="G$1" pin="(PCINT2/AIN1/ADC2)PA2"/>
+<pinref part="SW1" gate="G$1" pin="11"/>
+<wire x1="58.42" y1="71.12" x2="88.9" y2="71.12" width="0.1524" layer="91"/>
+<wire x1="88.9" y1="71.12" x2="88.9" y2="48.26" width="0.1524" layer="91"/>
+</segment>
+</net>
+<net name="N$4" class="0">
+<segment>
+<pinref part="U$1" gate="G$1" pin="(PCINT3/T0/ADC3)PA3"/>
+<pinref part="SW1" gate="G$1" pin="12"/>
+<wire x1="58.42" y1="73.66" x2="83.82" y2="73.66" width="0.1524" layer="91"/>
+<wire x1="83.82" y1="73.66" x2="83.82" y2="48.26" width="0.1524" layer="91"/>
+</segment>
+</net>
+<net name="N$16" class="0">
+<segment>
+<pinref part="U$1" gate="G$1" pin="(PCINT7/ICP/OC0B/ADC7)PA7"/>
+<pinref part="SW1" gate="G$1" pin="16"/>
+<wire x1="58.42" y1="83.82" x2="63.5" y2="83.82" width="0.1524" layer="91"/>
+<wire x1="63.5" y1="83.82" x2="63.5" y2="48.26" width="0.1524" layer="91"/>
+</segment>
+</net>
