File: Lokomotiv/schematics/LokomotivRevB.brd (EAGLE design)
At the start: 74.6 x 53.3 mm, 24 parts

Commit message: More pinne fix and circuit stuff
Other:
- board text added: "Lokomotiv Rev3"
- board text removed: "Lokomotov RevB"
Changed lines of the file:
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@@
 <hole x="71.12" y="49.53" drill="1.3"/>
 <hole x="71.12" y="3.81" drill="1.3"/>
-<text x="11.43" y="20.32" size="1.778" layer="1">Lokomotov
-RevB</text>
+<text x="11.43" y="20.32" size="1.778" layer="1">Lokomotiv
+Rev3</text>
 </plain>
 <attributes>
@@
 </variantdefs>
 <classes>
-<class number="0" name="Default" width="0.2032" drill="0.381">
-<clearance class="0" value="0.635"/>
+<class number="0" name="Default" width="0.4064" drill="0.381">
+<clearance class="0" value="1.016"/>
 </class>
 <class number="1" name="vcc" width="0" drill="0">
@@
 <via x="54.61" y="16.51" extent="1-16" drill="1.3" shape="square"/>
 <via x="46.99" y="36.83" extent="1-16" drill="1.3" shape="square"/>
+<wire x1="71.755" y1="42.275" x2="71.96" y2="30.59" width="0" layer="19" extent="1-1"/>
 </signal>
 <signal name="VCC">
@@
 <wire x1="54.61" y1="45.72" x2="54.61" y2="43.18" width="1.016" layer="16"/>
 <wire x1="12.7" y1="38.1" x2="8.89" y2="38.1" width="1.016" layer="16"/>
-<via x="8.89" y="38.1" extent="1-16" drill="0.6" shape="square"/>
+<via x="8.89" y="38.1" extent="1-16" drill="1.3" shape="square"/>
 <wire x1="8.89" y1="38.1" x2="7.62" y2="39.37" width="1.016" layer="1"/>
 <wire x1="7.62" y1="39.37" x2="7.62" y2="40.91" width="1.016" layer="1"/>

Commit message: EnkelFugl and some circuit changes
Parts:
- added JP1: (no value), SparkFun-Connectors:1X06
- added JP2: (no value), SparkFun-Connectors:1X05
- added JP3: M01PTH, SparkFun-Connectors:1X01
- moved R4 7.10 mm to (61.0, 33.7), turned to 270 degrees
- moved HALLENCODER 2.84 mm to (49.5, 41.9)
- moved VNH5019 2.54 mm to (39.4, 24.1)
- moved R7 2.54 mm to (10.2, 39.4)
- moved R8 2.54 mm to (7.62, 39.4)
- moved IRRECV 1.27 mm to (39.4, 41.9)
Connections:
- new net N$10: JP1.5, LEO_A[0..5].5
- new net N$11: JP1.4, LEO_A[0..5].4
- new net N$12: JP1.3, LEO_A[0..5].3
- new net N$13: JP1.2, LEO_A[0..5].2
- new net N$14: JP1.1, LEO_A[0..5].1
- new net N$15: JP2.5, LEO[0..7].5
- new net N$16: JP2.4, LEO[0..7].4
- new net N$17: JP2.3, LEO[0..7].3
- new net N$18: JP2.2, LEO[0..7].2
- new net N$19: JP2.1, LEO[0..7].1
- new net N$20: JP3.1, LEO8_13.9
- new net N$8: JP1.6, LEO_A[0..5].6
- new net N$9: LED4.C, LEO[0..7].7, R4.1
- net TX: now also R4.2; no longer LED4.C, LEO[0..7].7, R4.1
- net VCC: no longer R4.2
Routing:
- net TX: track 44.1 -> 24.8 mm
- net N$9: track 0.00 -> 16.4 mm
- net HALLIN: track 12.5 -> 17.4 mm
- net N$8: track 0.00 -> 3.81 mm
- net N$14: track 0.00 -> 3.81 mm
- net N$13: track 0.00 -> 3.81 mm
- net N$12: track 0.00 -> 3.81 mm
- net N$11: track 0.00 -> 3.81 mm
- net N$10: track 0.00 -> 3.81 mm
- net N$20: track 0.00 -> 3.28 mm
- net N$19: track 0.00 -> 3.17 mm
- net N$18: track 0.00 -> 3.17 mm
- net N$17: track 0.00 -> 3.17 mm
- net N$16: track 0.00 -> 3.17 mm
- net N$15: track 0.00 -> 3.17 mm
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Other:
- board text added: "Lokomotiv RevB"
- board text removed: "Lokomotiv Rev3"
