File: Lokomotiv/schematics/LokomotivRevB.sch (EAGLE design)
At the start: 24 parts

Commit message: EnkelFugl and some circuit changes
Parts:
- added JP1: (no value), SparkFun-Connectors:M06SIP
- added JP2: (no value), SparkFun-Connectors:M05PTH
- added JP3: M01PTH, SparkFun-Connectors:M01PTH
Connections:
- new net N$10: JP1.5, LEO_A[0..5].5
- new net N$11: JP1.4, LEO_A[0..5].4
- new net N$12: JP1.3, LEO_A[0..5].3
- new net N$13: JP1.2, LEO_A[0..5].2
- new net N$14: JP1.1, LEO_A[0..5].1
- new net N$15: JP2.5, LEO[0..7].5
- new net N$16: JP2.4, LEO[0..7].4
- new net N$17: JP2.3, LEO[0..7].3
- new net N$18: JP2.2, LEO[0..7].2
- new net N$19: JP2.1, LEO[0..7].1
- new net N$20: JP3.1, LEO8_13.9
- new net N$8: JP1.6, LEO_A[0..5].6
- new net N$9: LED4.C, LEO[0..7].7, R4.1
- net TX: now also R4.2; no longer LED4.C, LEO[0..7].7, R4.1
- net VCC: no longer R4.2
Other:
- moved on the sheet: R3, R4
Changed lines of the file:
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@@
 <part name="SUPPLY7" library="SparkFun-Aesthetics" deviceset="VCC" device=""/>
 <part name="GND8" library="SparkFun-Aesthetics" deviceset="GND" device=""/>
-<part name="SUPPLY8" library="SparkFun-Aesthetics" deviceset="VCC" device=""/>
 <part name="SUPPLY9" library="SparkFun-Aesthetics" deviceset="VCC" device=""/>
 <part name="GND9" library="SparkFun-Aesthetics" deviceset="GND" device=""/>
@@
 <part name="R9" library="adafruit" deviceset="R-US_" device="R0805" value="1K"/>
 <part name="R10" library="adafruit" deviceset="R-US_" device="R0805" value="1K"/>
+<part name="JP1" library="SparkFun-Connectors" deviceset="M06" device="SIP"/>
+<part name="JP2" library="SparkFun-Connectors" deviceset="M05" device="PTH"/>
+<part name="JP3" library="SparkFun-Connectors" deviceset="M01" device="PTH"/>
 </parts>
 <sheets>
@@
 <instance part="R2" gate="G$1" x="-81.28" y="50.8" rot="R90"/>
 <instance part="Q1" gate="G$1" x="-66.04" y="99.06"/>
-<instance part="R3" gate="G$1" x="-48.26" y="86.36" rot="R90"/>
-<instance part="R4" gate="G$1" x="-48.26" y="96.52" rot="R90"/>
+<instance part="R3" gate="G$1" x="-50.8" y="86.36" rot="R90"/>
+<instance part="R4" gate="G$1" x="-43.18" y="91.44" rot="R180"/>
 <instance part="SUPPLY4" gate="1" x="-63.5" y="124.46"/>
-<instance part="GND5" gate="1" x="-48.26" y="76.2"/>
+<instance part="GND5" gate="1" x="-50.8" y="76.2"/>
 <instance part="R5" gate="G$1" x="-73.66" y="88.9" rot="R90"/>
 <instance part="R6" gate="G$1" x="-63.5" y="114.3" rot="R90"/>
@@
 <instance part="SUPPLY7" gate="1" x="101.6" y="78.74" rot="MR0"/>
 <instance part="GND8" gate="1" x="101.6" y="63.5" rot="MR0"/>
-<instance part="SUPPLY8" gate="1" x="-48.26" y="101.6"/>
 <instance part="SUPPLY9" gate="1" x="-17.78" y="27.94" rot="MR0"/>
 <instance part="GND9" gate="1" x="2.54" y="-2.54" rot="MR0"/>
@@
 <instance part="R9" gate="G$1" x="-30.48" y="111.76" rot="R90"/>
 <instance part="R10" gate="G$1" x="-22.86" y="111.76" rot="R90"/>
+<instance part="JP1" gate="G$1" x="50.8" y="88.9" rot="MR0"/>
+<instance part="JP2" gate="G$1" x="7.62" y="81.28" rot="MR0"/>
+<instance part="JP3" gate="G$1" x="7.62" y="66.04" rot="MR0"/>
 </instances>
 <busses>
@@
 <pinref part="R3" gate="G$1" pin="1"/>
 <pinref part="GND5" gate="1" pin="GND"/>
-<wire x1="-48.26" y1="81.28" x2="-48.26" y2="78.74" width="0.1524" layer="91"/>
+<wire x1="-50.8" y1="78.74" x2="-50.8" y2="81.28" width="0.1524" layer="91"/>
 </segment>
 <segment>
@@
 <pinref part="LEO_VIN_GND" gate="1" pin="5"/>
 <wire x1="35.56" y1="66.04" x2="48.26" y2="66.04" width="0.1524" layer="91"/>
-</segment>
-<segment>
-<pinref part="R4" gate="G$1" pin="2"/>
-<pinref part="SUPPLY8" gate="1" pin="VCC"/>
 </segment>
 <segment>
@@
 <net name="TX" class="0">
 <segment>
-<pinref part="R4" gate="G$1" pin="1"/>
+<pinref part="XB1" gate="G$1" pin="DIN/!CONFIG"/>
+<label x="-93.98" y="81.28" size="1.778" layer="95"/>
+<pinref part="R4" gate="G$1" pin="2"/>
+<wire x1="-58.42" y1="81.28" x2="-96.52" y2="81.28" width="0.1524" layer="91"/>
+<wire x1="-48.26" y1="91.44" x2="-50.8" y2="91.44" width="0.1524" layer="91"/>
+<wire x1="-50.8" y1="91.44" x2="-58.42" y2="91.44" width="0.1524" layer="91"/>
+<wire x1="-58.42" y1="91.44" x2="-58.42" y2="81.28" width="0.1524" layer="91"/>
 <pinref part="R3" gate="G$1" pin="2"/>
-<junction x="-48.26" y="91.44"/>
-<wire x1="-48.26" y1="91.44" x2="-55.88" y2="91.44" width="0.1524" layer="91"/>
-<wire x1="-55.88" y1="91.44" x2="-55.88" y2="81.28" width="0.1524" layer="91"/>
-<pinref part="XB1" gate="G$1" pin="DIN/!CONFIG"/>
-<wire x1="-55.88" y1="81.28" x2="-96.52" y2="81.28" width="0.1524" layer="91"/>
-<label x="-45.72" y="91.44" size="1.778" layer="95"/>
-<label x="-93.98" y="81.28" size="1.778" layer="95"/>
-<wire x1="-48.26" y1="91.44" x2="-22.86" y2="91.44" width="0.1524" layer="91"/>
-<pinref part="LEO[0..7]" gate="1" pin="7"/>
-<pinref part="LED4" gate="G$1" pin="C"/>
-<wire x1="-22.86" y1="91.44" x2="-12.7" y2="91.44" width="0.1524" layer="91"/>
-<wire x1="-22.86" y1="99.06" x2="-22.86" y2="91.44" width="0.1524" layer="91"/>
-<junction x="-22.86" y="91.44"/>
+<junction x="-50.8" y="91.44"/>
 </segment>
 </net>
@@
 </segment>
 </net>
+<net name="N$9" class="0">
+<segment>
+<pinref part="LEO[0..7]" gate="1" pin="7"/>
+<wire x1="-22.86" y1="91.44" x2="-12.7" y2="91.44" width="0.1524" layer="91"/>
+<pinref part="LED4" gate="G$1" pin="C"/>
+<wire x1="-22.86" y1="99.06" x2="-22.86" y2="91.44" width="0.1524" layer="91"/>
+<wire x1="-38.1" y1="91.44" x2="-22.86" y2="91.44" width="0.1524" layer="91"/>
+<junction x="-22.86" y="91.44"/>
+<pinref part="R4" gate="G$1" pin="1"/>
+</segment>
+</net>
+<net name="N$8" class="0">
+<segment>
+<pinref part="LEO_A[0..5]" gate="1" pin="6"/>
+<wire x1="35.56" y1="96.52" x2="45.72" y2="96.52" width="0.1524" layer="91"/>
+<pinref part="JP1" gate="G$1" pin="6"/>
+</segment>
+</net>
+<net name="N$10" class="0">
+<segment>
+<pinref part="LEO_A[0..5]" gate="1" pin="5"/>
+<wire x1="35.56" y1="93.98" x2="45.72" y2="93.98" width="0.1524" layer="91"/>
+<pinref part="JP1" gate="G$1" pin="5"/>
+</segment>
+</net>
+<net name="N$11" class="0">
+<segment>
+<pinref part="LEO_A[0..5]" gate="1" pin="4"/>
+<wire x1="35.56" y1="91.44" x2="45.72" y2="91.44" width="0.1524" layer="91"/>
+<pinref part="JP1" gate="G$1" pin="4"/>
+</segment>
+</net>
+<net name="N$12" class="0">
+<segment>
+<pinref part="LEO_A[0..5]" gate="1" pin="3"/>
+<wire x1="35.56" y1="88.9" x2="45.72" y2="88.9" width="0.1524" layer="91"/>
+<pinref part="JP1" gate="G$1" pin="3"/>
+</segment>
+</net>
+<net name="N$13" class="0">
+<segment>
+<pinref part="LEO_A[0..5]" gate="1" pin="2"/>
+<wire x1="35.56" y1="86.36" x2="45.72" y2="86.36" width="0.1524" layer="91"/>
+<pinref part="JP1" gate="G$1" pin="2"/>
+</segment>
+</net>
+<net name="N$14" class="0">
+<segment>
+<pinref part="LEO_A[0..5]" gate="1" pin="1"/>
+<wire x1="35.56" y1="83.82" x2="45.72" y2="83.82" width="0.1524" layer="91"/>
+<pinref part="JP1" gate="G$1" pin="1"/>
+</segment>
+</net>
+<net name="N$15" class="0">
+<segment>
+<pinref part="LEO[0..7]" gate="1" pin="5"/>
+<pinref part="JP2" gate="G$1" pin="5"/>
+<wire x1="-12.7" y1="86.36" x2="0" y2="86.36" width="0.1524" layer="91"/>
+</segment>
+</net>
+<net name="N$16" class="0">
+<segment>
+<pinref part="LEO[0..7]" gate="1" pin="4"/>
+<pinref part="JP2" gate="G$1" pin="4"/>
+<wire x1="-12.7" y1="83.82" x2="0" y2="83.82" width="0.1524" layer="91"/>
+</segment>
+</net>
+<net name="N$17" class="0">
+<segment>
+<pinref part="LEO[0..7]" gate="1" pin="3"/>
+<pinref part="JP2" gate="G$1" pin="3"/>
+<wire x1="-12.7" y1="81.28" x2="0" y2="81.28" width="0.1524" layer="91"/>
+</segment>
+</net>
+<net name="N$18" class="0">
+<segment>
+<pinref part="LEO[0..7]" gate="1" pin="2"/>
+<pinref part="JP2" gate="G$1" pin="2"/>
+<wire x1="-12.7" y1="78.74" x2="0" y2="78.74" width="0.1524" layer="91"/>
+</segment>
+</net>
+<net name="N$19" class="0">
+<segment>
+<pinref part="LEO[0..7]" gate="1" pin="1"/>
+<pinref part="JP2" gate="G$1" pin="1"/>
+<wire x1="-12.7" y1="76.2" x2="0" y2="76.2" width="0.1524" layer="91"/>
+</segment>
+</net>
+<net name="N$20" class="0">
+<segment>
+<pinref part="LEO8_13" gate="1" pin="9"/>
+<pinref part="JP3" gate="G$1" pin="1"/>
+<wire x1="-12.7" y1="66.04" x2="0" y2="66.04" width="0.1524" layer="91"/>
+</segment>
+</net>
