File: ServoMega/schematics/ServoCity.sch (EAGLE design)
At the start: 2 parts

Commit message: HOK post laptop update
Parts:
- added C1, C2, C3, C4: (no value), rcl:C-EUC0805
- added C5: 2k2, rcl:CPOL-EUE10-20
- added C6: 470, rcl:CPOL-EUE5-10.5
- added C8, C9: (no value), eagle-ltspice:C
- added IC1: MAX232, maxim:MAX232
- added S10, S11, S12, S13, S14, S15, S16, S17, S18, S19, S2, S20, S21, S22, S23, S24, S25, S26, S27, S28, S29, S3, S30, S31, S32, S4, S5, S6, S7, S8, S9: 22-23-2031, con-molex:22-23-2031
- added X1: (no value), con-molex:KK-156-2
- added X2: (no value), con-molex:KK-156-3
Connections:
- new net 5V: C5.+, C6.+, C8.1, C9.1, S1-2.S, S10-2.S, S11-2.S, S12-2.S, S13-2.S, S14-2.S, S15-2.S, S16-2.S, S17-2.S, S18-2.S, S19-2.S, S2-2.S, S20-2.S, S21-2.S, S22-2.S, S23-2.S, S24-2.S, S25-2.S, S26-2.S, S27-2.S, S28-2.S, S29-2.S, S3-2.S, S30-2.S, S31-2.S, S32-2.S, S4-2.S, S5-2.S, S6-2.S, S7-2.S, S8-2.S, S9-2.S, X1-1.S
- new net GND: C4.2, C5.-, C6.-, C8.2, C9.2, S1-3.S, S10-3.S, S11-3.S, S12-3.S, S13-3.S, S14-3.S, S15-3.S, S16-3.S, S17-3.S, S18-3.S, S19-3.S, S2-3.S, S20-3.S, S21-3.S, S22-3.S, S23-3.S, S24-3.S, S25-3.S, S26-3.S, S27-3.S, S28-3.S, S29-3.S, S3-3.S, S30-3.S, S31-3.S, S32-3.S, S4-3.S, S5-3.S, S6-3.S, S7-3.S, S8-3.S, S9-3.S, U$1.5V_ICSP, U$1.GND1, U$1.GND_1, U$1.GND_2, U$1.GND_A, U$1.GND_B, X1-2.S, X2-1.S
- new net N$1: IC1G$1.T1OUT, X2-2.S
- new net N$2: IC1G$1.R1IN, X2-3.S
- new net N$3: C1.1, IC1G$1.C1+
- new net N$4: C1.2, IC1G$1.C1-
- new net N$5: C2.1, IC1G$1.C2+
- new net N$6: C2.2, IC1G$1.C2-
- new net N$7: C3.1, IC1G$1.V+
- new net N$8: C3.2, IC1G$1.V-
- new net RX: IC1G$1.R1OUT, U$1.RX0
- new net SERVO1: S1-1.S, U$1.23
- new net SERVO10: S10-1.S, U$1.41
- new net SERVO11: S11-1.S, U$1.43
- new net SERVO12: S12-1.S, U$1.45
- new net SERVO13: S13-1.S, U$1.47
- new net SERVO14: S14-1.S, U$1.49
- new net SERVO15: S15-1.S, U$1.51
- new net SERVO16: S16-1.S, U$1.53
- new net SERVO17: S17-1.S, U$1.22
- new net SERVO18: S18-1.S, U$1.24
- new net SERVO19: S19-1.S, U$1.26
- new net SERVO2: S2-1.S, U$1.25
- new net SERVO20: S20-1.S, U$1.28
- new net SERVO21: S21-1.S, U$1.30
- new net SERVO22: S22-1.S, U$1.32
- new net SERVO23: S23-1.S, U$1.34
- new net SERVO24: S24-1.S, U$1.36
- new net SERVO25: S25-1.S, U$1.38
- new net SERVO26: S26-1.S, U$1.40
- new net SERVO27: S27-1.S, U$1.42
- new net SERVO28: S28-1.S, U$1.44
- new net SERVO29: S29-1.S, U$1.46
- new net SERVO3: S3-1.S, U$1.27
- new net SERVO30: S30-1.S, U$1.48
- new net SERVO31: S31-1.S, U$1.50
- new net SERVO32: S32-1.S, U$1.52
- new net SERVO4: S4-1.S, U$1.29
- new net SERVO5: S5-1.S, U$1.31
- new net SERVO6: S6-1.S, U$1.33
- new net SERVO7: S7-1.S, U$1.35
- new net SERVO8: S8-1.S, U$1.37
- new net SERVO9: S9-1.S, U$1.39
- new net TX: IC1G$1.T1IN, U$1.TX0
- new net VCC: C4.1, U$1.5V, U$1.5V_A, U$1.5V_B, U$1.GND_ICSP
Other:
- moved on the sheet: S1-1, S1-2, S1-3
